File: type-A/kicad-files/type-A-pcb/type-A-pcb.kicad_sch (KiCad schematic)
At the start: 20 parts, among them J1 OLED-128x64, SW10 SW_Push, SW11 SW_Push, SW12 SW_Push, SW13 SW_Push, SW14 SW_Push, SW15 SW_Push, SW16 SW_Push, SW17 SW_Push, SW18 SW_Push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

Commit message: New Kicad library.
Parts:
- A1: renamed from SW15; footprint Switches Kailh:SW_Kailh_Choc_V1_1.00u -> kailh-pretty:Kailh_socket_PG1350_optional
- B1: renamed from SW13; footprint Switches Kailh:SW_Kailh_Choc_V1_1.00u -> kailh-pretty:Kailh_socket_PG1350_optional
- Back1: renamed from SW18; footprint Switches Kailh:SW_Kailh_Choc_V1_1.00u -> kailh-pretty:Kailh_socket_PG1350_optional
- Down1: renamed from SW14; footprint Switches Kailh:SW_Kailh_Choc_V1_1.00u -> kailh-pretty:Kailh_socket_PG1350_optional
- LB1: renamed from SW5; footprint Switches Kailh:SW_Kailh_Choc_V1_1.00u -> kailh-pretty:Kailh_socket_PG1350_optional
- LT1: renamed from SW9; footprint Switches Kailh:SW_Kailh_Choc_V1_1.00u -> kailh-pretty:Kailh_socket_PG1350_optional
- Left1: renamed from SW10; footprint Switches Kailh:SW_Kailh_Choc_V1_1.00u -> kailh-pretty:Kailh_socket_PG1350_optional
- Option_1: renamed from L3; footprint Switches Kailh:SW_Kailh_Choc_V1_1.00u -> kailh-pretty:Kailh_socket_PG1350_optional
- Option_2: renamed from R3; footprint Switches Kailh:SW_Kailh_Choc_V1_1.00u -> kailh-pretty:Kailh_socket_PG1350_optional
- Option_3: renamed from SW3; footprint Switches Kailh:SW_Kailh_Choc_V1_1.00u -> kailh-pretty:Kailh_socket_PG1350_optional
- Option_4: renamed from SW4; footprint Switches Kailh:SW_Kailh_Choc_V1_1.00u -> kailh-pretty:Kailh_socket_PG1350_optional
- RB1: renamed from SW6; footprint Switches Kailh:SW_Kailh_Choc_V1_1.00u -> kailh-pretty:Kailh_socket_PG1350_optional
- RT1: renamed from SW11; footprint Switches Kailh:SW_Kailh_Choc_V1_1.00u -> kailh-pretty:Kailh_socket_PG1350_optional
- Right1: renamed from SW12; footprint Switches Kailh:SW_Kailh_Choc_V1_1.00u -> kailh-pretty:Kailh_socket_PG1350_optional
- Start1: renamed from SW17; footprint Switches Kailh:SW_Kailh_Choc_V1_1.00u -> kailh-pretty:Kailh_socket_PG1350_optional
- U1: footprint mcu-pretty:rp2040-zero-tht -> rp2040-zero-pretty:Waveshare_RP2040-Zero_TH
- Up1: renamed from SW16; footprint Switches Kailh:SW_Kailh_Choc_V1_1.00u -> kailh-pretty:Kailh_socket_PG1350_optional
- X1: renamed from SW8; footprint Switches Kailh:SW_Kailh_Choc_V1_1.00u -> kailh-pretty:Kailh_socket_PG1350_optional
- Y1: renamed from SW7; footprint Switches Kailh:SW_Kailh_Choc_V1_1.00u -> kailh-pretty:Kailh_socket_PG1350_optional
